Commit message: Yolo testing and Multicontroller

File: Arm_Urdf/urdf/Arm_Urdf.urdf (robot description, URDF)
Before this commit: robot Arm_Urdf, 15 links, 14 joints
Links:
- removed link camera_link_base_left
- removed link camera_link_base_right
- removed link camera_link_optical_base_left
- removed link camera_link_optical_base_right
Joints:
- removed joint camera_base_joint_right
- removed joint camera_joint_base_left
- removed joint camera_optical_joint_base_left
- removed joint camera_optical_joint_base_right
